File: pcb_codespace/TECHIN514_final/TECHIN514_final.kicad_pcb (KiCad board)
At the start: 2 copper layers, 68 x 45.7 mm, 5 parts, among them J1 Conn_01x02_Pin, U1 XIAO_ESP32_C3

Commit message: pcb_upload
Parts:
- added J2: Conn_01x02_Pin, Connector_PinHeader_1.00mm:PinHeader_1x02_P1.00mm_Vertical, F.Cu at (101.5, 103.5)
- added REF**: MountingHole_2.2mm_M2, MountingHole:MountingHole_2.2mm_M2, F.Cu at (58.5, 75.0)
- added REF**: MountingHole_2.2mm_M2, MountingHole:MountingHole_2.2mm_M2, F.Cu at (113.0, 75.0)
- added REF**: MountingHole_2.2mm_M2, MountingHole:MountingHole_2.2mm_M2, F.Cu at (85.5, 111.5)
Connections:
- U1 pad 16: Net-(J1-Pin_1) -> Net-(J2-Pin_1)
Routing:
- net Net-(J2-Pin_1): track 0.00 -> 5.78 mm
- net Net-(J1-Pin_1): track 12.7 -> 10.9 mm
