File: pcb_codespace/TECHIN514_final/TECHIN514_final.kicad_sch (KiCad schematic)
At the start: 14 parts, among them M1 Motor_DC

Commit message: lab 4
Parts:
- added BAT3: ~, symbol my_pcb:Battery
- added ESP3: ~, symbol my_pcb:XIAO_ESP32C3
- added R3: 1MΩ, symbol Device:R
- added RP2: ~, symbol my_pcb:RP-C18.3-ST
Connections:
- net at ESP2. (D7): now also BAT2. (-); no longer TB1. (BO1)
- net at ESP1. (D7): now also R2.2; no longer BAT1. (-)
- net at ESP1. (D7), RP1.: now also R2.1
- new net: BAT3. (-), ESP3. (D7) (x2)
- new net: ESP2. (D7), TB1. (BO1) (x4)
- new net: ESP3. (D7), RP2.
- new net: ESP3. (D7), R3.1, RP2.
- new net: ESP3. (D7), R3.2
- new net: BAT1. (-), ESP1. (D7)
- new net: BAT2. (-), ESP2. (D7)
- new net: ESP1. (D7), RP1.

Commit message: submission
Parts:
- removed BAT1, BAT2, BAT3: ~, symbol my_pcb:Battery
- removed C1, C3: 0.1uF, symbol Device:C
- removed C2, C4: 10uF, symbol Device:C_Polarized
- removed ESP1, ESP2, ESP3: ~, symbol my_pcb:XIAO_ESP32C3
- removed M1: Motor_DC, symbol Motor:Motor_DC
- removed R2, R3: 1MΩ, symbol Device:R
- removed RP1, RP2: ~, symbol my_pcb:RP-C18.3-ST
- removed TB1: ~, symbol my_pcb:TB6612FNG
- added J1: Conn_01x02_Pin, Connector_PinHeader_1.00mm:PinHeader_1x02_P1.00mm_Vertical, symbol Connector:Conn_01x02_Pin
- added U1: XIAO_ESP32_C3, Library:XIAO_ESP32, symbol my_pcb:XIAO_ESP32
- added stepper_motor1: x27 stepper motor, Library:x27_stepper, symbol my_pcb:x27stepper
- D1: value LED -> LSR976; footprint (none) -> LED_SMD:LED_0805_2012Metric_Pad1.15x1.40mm_HandSolder
- R1: value R -> 330Ω; footprint (none) -> Resistor_SMD:R_0603_1608Metric_Pad0.98x0.95mm_HandSolder
Connections:
- net GND: now reaches D1.1 (K)
- net GND: now also U1.13 (GND)
- net at R1.2: now also U1.7 (GPIO43_TX_D6)
- new net: J1.1 (Pin_1), U1.16 (-BATT)
- new net: J1.2 (Pin_2), U1.15 (+BATT)
- new net: U1.1 (GPIO1_A0_D0), stepper_motor1.1 (pin1)
- new net: U1.2 (GPIO2_A1_D1), stepper_motor1.2 (pin2)
- new net: U1.3 (GPIO3_A2_D2), stepper_motor1.3 (pin3)
- new net: U1.4 (GPIO4_A3_D3), stepper_motor1.4 (pin4)
Other:
- title: (none) -> Warren's PCB

Commit message: pcb_upload
Parts:
- added J2: Conn_01x02_Pin, Connector_PinHeader_1.00mm:PinHeader_1x02_P1.00mm_Vertical, symbol Connector:Conn_01x02_Pin
Connections:
- net at J1.1 (Pin_1): now also J2.2 (Pin_2); no longer U1.16 (-BATT)
- new net: J2.1 (Pin_1), U1.16 (-BATT)
Changed lines of the file:
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@@
 	)
 	(junction
-		(at 161.29 157.48)
+		(at 142.24 157.48)
 		(diameter 0)
 		(color 0 0 0 0)
@@
 	(wire
 		(pts
-			(xy 245.11 102.87) (xy 157.48 102.87)
+			(xy 245.11 102.87) (xy 189.23 102.87)
+		)
+		(stroke
+			(width 0)
+			(type default)
+		)
+	)
+	(wire
+		(pts
+			(xy 186.69 99.06) (xy 186.69 102.87)
 		)
 		(stroke
@@
 	(wire
 		(pts
+			(xy 189.23 99.06) (xy 189.23 102.87)
+		)
+		(stroke
+			(width 0)
+			(type default)
+		)
+	)
+	(wire
+		(pts
 			(xy 184.15 127) (xy 190.5 127)
 		)
@@
 	(wire
 		(pts
-			(xy 161.29 157.48) (xy 161.29 163.83)
+			(xy 142.24 157.48) (xy 142.24 165.1)
 		)
 		(stroke
@@
 	(wire
 		(pts
-			(xy 102.87 157.48) (xy 161.29 157.48)
+			(xy 142.24 157.48) (xy 161.29 157.48)
+		)
+		(stroke
+			(width 0)
+			(type default)
+		)
+	)
+	(wire
+		(pts
+			(xy 102.87 157.48) (xy 142.24 157.48)
+		)
+		(stroke
+			(width 0)
+			(type default)
+		)
+	)
+	(wire
+		(pts
+			(xy 186.69 102.87) (xy 157.48 102.87)
 		)
 		(stroke
@@
 	)
 	(symbol
+		(lib_id "Connector:Conn_01x02_Pin")
+		(at 189.23 93.98 270)
+		(unit 1)
+		(exclude_from_sim no)
+		(in_bom yes)
+		(on_board yes)
+		(dnp no)
+		(fields_autoplaced yes)
+		(property "Reference" "J2"
+			(at 190.5 93.3449 90)
+			(effects
+				(font
+					(size 1.27 1.27)
+				)
+				(justify left)
+			)
+		)
+		(property "Value" "Conn_01x02_Pin"
+			(at 190.5 95.8849 90)
+			(effects
+				(font
+					(size 1.27 1.27)
+				)
+				(justify left)
+			)
+		)
+		(property "Footprint" "Connector_PinHeader_1.00mm:PinHeader_1x02_P1.00mm_Vertical"
+			(at 189.23 93.98 0)
+			(effects
+				(font
+					(size 1.27 1.27)
+				)
+				(hide yes)
+			)
+		)
+		(property "Datasheet" "~"
+			(at 189.23 93.98 0)
+			(effects
+				(font
+					(size 1.27 1.27)
+				)
+				(hide yes)
+			)
+		)
+		(property "Description" "Generic connector, single row, 01x02, script generated"
+			(at 189.23 93.98 0)
+			(effects
+				(font
+					(size 1.27 1.27)
+				)
+				(hide yes)
+			)
+		)
+		(pin "1"
+		)
+		(pin "2"
+		)
+		(instances
+			(project "TECHIN514_final"
+				(path "/e6281833-f3ff-436e-9d5d-e5d1fca3e81a"
+					(reference "J2")
+					(unit 1)
+				)
+			)
+		)
+	)
+	(symbol
 		(lib_id "Device:LED")
 		(at 111.76 142.24 0)
@@
 	(symbol
 		(lib_id "power:GND")
-		(at 161.29 163.83 0)
+		(at 142.24 165.1 0)
 		(unit 1)
 		(exclude_from_sim no)
@@
 		(fields_autoplaced yes)
 		(property "Reference" "#PWR01"
-			(at 161.29 170.18 0)
+			(at 142.24 171.45 0)
 			(effects
 				(font
@@
 		)
 		(property "Value" "GND"
-			(at 161.29 168.91 0)
+			(at 142.24 170.18 0)
 			(effects
 				(font
@@
 		)
 		(property "Footprint" ""
-			(at 161.29 163.83 0)
+			(at 142.24 165.1 0)
 			(effects
 				(font
@@
 		)
 		(property "Datasheet" ""
-			(at 161.29 163.83 0)
+			(at 142.24 165.1 0)
 			(effects
 				(font
@@
 		)
 		(property "Description" "Power symbol creates a global label with name \"GND\" , ground"
-			(at 161.29 163.83 0)
-			(effects
-				(font
+			(at 142.24 165.1 0)
+			(effects
+				(font
